File: aair_gimb_pcb/mosfet.kicad_sch (KiCad schematic)
At the start: 15 parts, among them Q1 sir182dp, Q2 sir182dp, Q3 sir182dp, Q4 sir182dp, Q5 sir182dp, Q6 sir182dp

Commit message: сделать коннектор для переыерии
Changed lines of the file:
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@@
 	)
 	(hierarchical_label "H3_LOW"
-		(shape input)
+		(shape output)
 		(at 180.34 119.38 270)
 		(effects
@@
 	)
 	(hierarchical_label "H2_LOW"
-		(shape input)
+		(shape output)
 		(at 146.05 119.38 270)
 		(effects
@@
 	)
 	(hierarchical_label "H1_LOW"
-		(shape input)
+		(shape output)
 		(at 110.49 119.38 270)
 		(effects
