File: aair_gimb_pcb/aair_gimb_pcb.kicad_pcb (KiCad board)
At the start: 4 copper layers, 95.5 x 42 mm, 90 parts, among them J1 I2C, J2 UART, J3 USB_B_Mini, J5 SWD, J6 SPI1, P3 A, P4 B, P5 C, Q1 sir182dp, Q2 sir182dp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

Commit message: fix exeption to pcb
Parts:
- C13, C14, C15, C16, C22, C27, C28, C29, C30, C31, C32, C33, C34, C35, C36, D1, U3: moved to B.Cu
- moved C36 78.0 mm to (174.0, 78.7), turned to 90 degrees
- moved C16 77.2 mm to (145.4, 70.7), turned to -90 degrees
- moved C14 76.3 mm to (146.9, 70.7), turned to -90 degrees
- moved C15 76.1 mm to (151.8, 70.8), turned to -90 degrees
- moved C13 76.0 mm to (150.2, 70.8), turned to -90 degrees
- moved R6 72.6 mm to (149.9, 79.3), turned to 180 degrees
- moved C1 70.5 mm to (152.9, 88.1), turned to 180 degrees
- moved C7 69.8 mm to (153.2, 80.4), turned to 180 degrees
- moved C35 66.3 mm to (171.2, 87.5), turned to 180 degrees
- moved C34 65.7 mm to (171.6, 85.1), turned to 180 degrees
- moved C33 64.0 mm to (170.1, 82.8), turned to 180 degrees
- moved C32 63.3 mm to (170.1, 80.3), turned to 180 degrees
- moved C31 62.6 mm to (170.1, 77.8), turned to 180 degrees
- moved C12 61.7 mm to (149.7, 81.7), turned to -90 degrees
- moved C4 59.8 mm to (149.3, 99.0), turned to -90 degrees
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Routing:
- net +3.3V: track 0.00 -> 136.3 mm, vias 0 -> 7
- net GND: track 139.9 -> 212.3 mm, vias 12 -> 15
- net /drv8302/H2_VS: track 69.3 -> 126.2 mm, vias 2 -> 4
- net /drv8302/H3_VS: track 87.3 -> 144.1 mm, vias 2 -> 3
- net +5V: track 0.00 -> 52.3 mm, vias 0 -> 3
- net NRST: track 0.00 -> 48.9 mm, vias 0 -> 3
- net V_SUPPLY: track 33.8 -> 75.3 mm, vias 2 -> 3
- net /Stm32f405/FAULT: track 0.00 -> 32.5 mm, vias 0 -> 2
- net /drv8302/H1_VS: track 86.1 -> 117.9 mm, vias 2 -> 3
- net /Stm32f405/EN_GATE: track 0.00 -> 28.0 mm, vias 0 -> 2
- net USB_D-: track 0.00 -> 26.7 mm, vias 0 -> 2
- net SWDIO: track 0.00 -> 24.9 mm, vias 0 -> 2
- net Net-(U2-BOOT0): track 0.00 -> 24.3 mm
- net USB_D+: track 0.00 -> 24.1 mm, vias 0 -> 2
- net SWCLK: track 0.00 -> 23.1 mm, vias 0 -> 2
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- added copper zone on F.Cu, net GND
- added copper zone on In1.Cu, net GND
- added copper zone on In2.Cu, net GND
Other:
- board size 95.5 x 42 mm -> 81.9 x 47.9 mm
