File: aair_gimb_pcb/aair_gimb_pcb.kicad_pcb (KiCad board)
At the start: 4 copper layers, 81.9 x 47.9 mm, 90 parts, among them J1 I2C, J2 UART, J3 USB_B_Mini, J5 SWD, J6 SPI1, P3 A, P4 B, P5 C, Q1 sir182dp, Q2 sir182dp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

Commit message: done
Parts:
- U1: footprint CRF1:TSSOP-56-PP -> Package_SO:HTSSOP-56-1EP_6.1x14mm_P0.5mm_EP3.61x6.35mm
- moved C26 8.09 mm to (165.1, 100.2), turned to 90 degrees
- moved R25 4.63 mm to (130.8, 79.2)
- moved C21 3.12 mm to (169.5, 90.5)
- moved C25 1.95 mm to (159.6, 100.8)
- moved C17 1.86 mm to (159.6, 98.3)
- moved C29 1.23 mm to (156.6, 67.5)
- moved R24 0.76 mm to (139.8, 79.8)
- moved D3 0.28 mm to (165.8, 76.7)
- moved C18 0.25 mm to (165.7, 83.0)
- moved U1 0.20 mm to (159.7, 88.2), turned to 0 degrees
- moved R1 0.19 mm to (145.8, 79.6)
- moved C20 0.06 mm to (167.3, 85.7)
- renumbered BOOT to B1, NR to NR1
Routing:
- net GND: track 212.3 -> 286.9 mm, vias 15 -> 30
- net Net-(U1-DVDD): track 11.9 -> 34.7 mm, vias 2 -> 3
- net V_SUPPLY: track 75.3 -> 83.3 mm, vias 3 -> 2
- net /drv8302/H2_LOW: track 65.2 -> 69.9 mm
- net /drv8302/H1_LOW: track 80.0 -> 84.6 mm
- net UART_TX: track 17.0 -> 21.4 mm
- net /Stm32f405/SENS2: track 13.0 -> 16.9 mm
- net Net-(U1-BST_C): track 2.00 -> 5.44 mm
- net VCC: track 21.0 -> 23.8 mm
- net /Stm32f405/L2: track 12.6 -> 15.2 mm
- net /Stm32f405/M_PWM: track 19.4 -> 17.5 mm
- net /drv8302/H2_VS: track 126.2 -> 127.8 mm
- net Net-(D3-K): track 15.4 -> 17.0 mm
- net /Stm32f405/H3: track 17.1 -> 18.7 mm
- net /Stm32f405/FAULT: track 32.5 -> 33.8 mm
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
Commit message: готово
Parts:
- added REF**: MountingHole_2.2mm_M2_ISO7380, MountingHole:MountingHole_2.2mm_M2_ISO7380, F.Cu at (125.3, 100.6)
- added REF**: MountingHole_2.2mm_M2_ISO7380, MountingHole:MountingHole_2.2mm_M2_ISO7380, F.Cu at (124.8, 62.5)
- added REF**: MountingHole_2.2mm_M2_ISO7380, MountingHole:MountingHole_2.2mm_M2_ISO7380, F.Cu at (200.8, 62.7)
- added REF**: MountingHole_2.2mm_M2_ISO7380, MountingHole:MountingHole_2.2mm_M2_ISO7380, F.Cu at (201.0, 100.8)
- renumbered P3 to A, P4 to B, P5 to C
Connections:
- J1 pad MP: (no net) -> GND
- J2 pad MP: (no net) -> GND
- J3 pad 6: unconnected-(J3-Shield-Pad6)_2 -> GND
- J5 pad MP: (no net) -> GND
- J6 pad MP: (no net) -> GND
Other:
- board size 81.9 x 47.9 mm -> 80.1 x 43 mm

Commit message: pcb, step
Routing:
- net V_SUPPLY: track 83.3 -> 81.4 mm
- net Net-(D3-K): track 17.0 -> 16.1 mm
Changed lines of the file:
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@@
 			(outputformat 1)
 			(mirror no)
-			(drillshape 1)
+			(drillshape 0)
 			(scaleselection 1)
-			(outputdirectory "")
+			(outputdirectory "pcb/")
 		)
 	)
@@
 			)
 		)
+		(model "C:/Users/Gigabyte/Downloads/amass-xt30pw-m-_-pcb-solder-1.snapshot.2/Amass_XT30PW-M_pcb solder.stp"
+			(offset
+				(xyz -2.5 4 2.5)
+			)
+			(scale
+				(xyz 1 1 1)
+			)
+			(rotate
+				(xyz -0 -0 -180)
+			)
+		)
 	)
 	(footprint "CRF1:SMD-0603_r"
@@
 	)
 	(segment
-		(start 162.49 82.99)
-		(end 163.4534 82.99)
+		(start 163.4534 94.99)
+		(end 162.01 94.99)
 		(width 0.2)
 		(layer "F.Cu")
@@
 	)
 	(segment
-		(start 163.4534 94.99)
-		(end 162.01 94.99)
-		(width 0.2)
+		(start 161.5 82)
+		(end 162.25 82.75)
+		(width 0.7)
 		(layer "F.Cu")
 		(net 2)
@@
 	)
 	(segment
-		(start 161.5 82)
-		(end 162.49 82.99)
-		(width 0.2)
-		(layer "F.Cu")
-		(net 2)
-	)
-	(segment
 		(start 163.4534 94.99)
 		(end 163.4534 96.4534)
@@
 	)
 	(segment
-		(start 161.5 82)
-		(end 161.99 82.49)
-		(width 0.2)
+		(start 162.25 82.75)
+		(end 163.85 82.75)
+		(width 0.7)
 		(layer "F.Cu")
 		(net 2)
@@
 	)
 	(segment
-		(start 161.99 82.49)
-		(end 163.4534 82.49)
-		(width 0.2)
-		(layer "F.Cu")
-		(net 2)
-	)
-	(segment
 		(start 162.55 100.85)
 		(end 161.025 100.85)
@@
 	)
 	(segment
+		(start 160.1005 83.4505)
+		(end 160.4 83.75)
+		(width 0.6)
+		(layer "F.Cu")
+		(net 17)
+	)
+	(segment
 		(start 163.4534 84.49)
 		(end 163.4044 84.539)
@@
 	)
 	(segment
-		(start 165.372 83.99)
-		(end 163.4534 83.99)
-		(width 0.2)
+		(start 161.95 84.2)
+		(end 163.65 84.2)
+		(width 0.6)
 		(layer "F.Cu")
 		(net 17)
 	)
 	(segment
-		(start 160.1005 79.85278)
-		(end 160.1005 81.20597)
-		(width 1)
+		(start 161.5 83.75)
+		(end 161.95 84.2)
+		(width 0.6)
 		(layer "F.Cu")
 		(net 17)
 	)
 	(segment
-		(start 161.74 83.99)
-		(end 160.1005 82.3505)
+		(start 165.372 83.99)
+		(end 163.4534 83.99)
 		(width 0.2)
 		(layer "F.Cu")
@@
 	)
 	(segment
-		(start 163.4044 84.539)
-		(end 162.289 84.539)
-		(width 0.2)
-		(layer "F.Cu")
-		(net 17)
-	)
-	(segment
-		(start 160.1005 82.3505)
-		(end 160.1005 81.20597)
-		(width 0.2)
+		(start 160.1005 83.4505)
+		(end 160.1005 79.85278)
+		(width 0.6)
 		(layer "F.Cu")
 		(net 17)
 	)
 	(segment
-		(start 162.289 84.539)
-		(end 161.74 83.99)
-		(width 0.2)
+		(start 160.4 83.75)
+		(end 161.5 83.75)
+		(width 0.6)
 		(layer "F.Cu")
 		(net 17)
@@
 	)
 	(segment
-		(start 163.4534 83.99)
-		(end 161.74 83.99)
-		(width 0.2)
-		(layer "F.Cu")
-		(net 17)
-	)
-	(segment
 		(start 193.88 79.48)
 		(end 196.5 79.48)
@@
 	)
 	(segment
+		(start 167.29 86.49)
+		(end 167.3 86.5)
+		(width 0.2)
+		(layer "F.Cu")
+		(net 21)
+	)
+	(segment
 		(start 168.560659 84.95)
 		(end 168.56066 84.950001)
@@
 	)
 	(segment
+		(start 163.4534 86.49)
+		(end 167.29 86.49)
+		(width 0.3)
+		(layer "F.Cu")
+		(net 21)
+	)
+	(segment
 		(start 193.865 69.02)
 		(end 195.72 69.02)
@@
 	)
 	(segment
+		(start 163.4534 86.49)
+		(end 163.4944 86.449)
+		(width 0.2)
+		(layer "F.Cu")
+		(net 21)
+	)
+	(segment
 		(start 168.56066 85.30134)
 		(end 167.3 86.562)
@@
 	)
 	(segment
-		(start 163.4944 86.449)
-		(end 167.249 86.449)
-		(width 0.2)
-		(layer "F.Cu")
-		(net 21)
-	)
-	(segment
-		(start 167.249 86.449)
-		(end 167.3 86.5)
-		(width 0.2)
-		(layer "F.Cu")
-		(net 21)
-	)
-	(segment
-		(start 163.4534 86.49)
-		(end 163.4944 86.449)
-		(width 0.2)
-		(layer "F.Cu")
-		(net 21)
-	)
-	(segment
 		(start 190.45 75.6)
 		(end 190.45 74.315)
@@
 	)
 	(segment
+		(start 167.249 86.449)
+		(end 167.3 86.5)
+		(width 0.2)
+		(layer "F.Cu")
+		(net 21)
+	)
+	(segment
 		(start 195.72 69.02)
 		(end 197.635 70.935)
@@
 	)
 	(segment
-		(start 163.4534 87.49)
-		(end 164.96 87.49)
+		(start 169.574 92.612)
+		(end 170.162 92.612)
 		(width 0.2)
 		(layer "F.Cu")
@@
 	)
 	(segment
-		(start 169.574 92.612)
-		(end 170.162 92.612)
+		(start 165.2 87.25)
+		(end 164.96 87.49)
 		(width 0.2)
 		(layer "F.Cu")
@@
 	)
 	(segment
+		(start 164.96 87.49)
+		(end 163.4534 87.49)
+		(width 0.2)
+		(layer "F.Cu")
+		(net 67)
+	)
+	(segment
 		(start 177.9 75.99853)
 		(end 177.9 76.85)
@@
 	)
 	(segment
-		(start 164.96 87.49)
-		(end 165.4 87.05)
+		(start 165.29 87.25)
+		(end 165.2 87.25)
 		(width 0.2)
 		(layer "F.Cu")
@@
 	)
 	(segment
+		(start 165.4 87.14)
+		(end 165.29 87.25)
+		(width 0.2)
+		(layer "F.Cu")
+		(net 67)
+	)
+	(segment
 		(start 188.56 73.48)
 		(end 188.565 73.475)
@@
 	)
 	(via
-		(at 165.4 87.05)
+		(at 165.4 87.14)
 		(size 0.6)
 		(drill 0.3)
@@
 	)
 	(segment
-		(start 187.15 76.3)
-		(end 187.15 73.48)
+		(start 184.9 78.55)
+		(end 187.15 76.3)
 		(width 0.5)
 		(layer "In2.Cu")
@@
 	)
 	(segment
-		(start 165.4 87.05)
-		(end 173.9 78.55)
+		(start 165.4 87.14)
+		(end 165.4 87.05)
 		(width 0.5)
 		(layer "In2.Cu")
@@
 	)
 	(segment
-		(start 184.9 78.55)
-		(end 187.15 76.3)
+		(start 187.15 76.3)
+		(end 187.15 73.48)
 		(width 0.5)
 		(layer "In2.Cu")
@@
 		(layer "In2.Cu")
 		(net 67)
+	)
+	(segment
+		(start 165.4 87.05)
+		(end 173.9 78.55)
+		(width 0.5)
+		(layer "In2.Cu")
+		(net 67)
